File: Wuerfel_Schaltplan/Wuerfel_Schaltplan.kicad_sch (KiCad schematic)
At the start: 21 parts, among them SW1 SW_Push, SW2 SW_Push

Commit message: Finish PCB design
Connections:
- no-connect marks 0 -> 20
Other:
- company: (none) -> Philipp Uhlendorf
- title: (none) -> Elektronischer Würfel
- moved on the sheet: R8, R9, SW2
Changed lines of the file:
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@@
 	(generator_version "10.0")
 	(paper "A4")
+	(title_block
+		(title "Elektronischer Würfel")
+		(date "2026-08-24")
+		(rev "1.0.0")
+		(company "Philipp Uhlendorf")
+	)
 	(junction
-		(at 228.6 86.36)
+		(at 237.49 85.09)
 		(diameter 0)
 		(color 0 0 0 0)
@@
 	)
 	(junction
-		(at 228.6 74.93)
-		(diameter 0)
-		(color 0 0 0 0)
-	)
-	(junction
-		(at 237.49 86.36)
+		(at 228.6 85.09)
 		(diameter 0)
 		(color 0 0 0 0)
@@
 	)
 	(junction
+		(at 228.6 73.66)
+		(diameter 0)
+		(color 0 0 0 0)
+	)
+	(junction
 		(at 152.4 54.61)
 		(diameter 0)
 		(color 0 0 0 0)
 	)
+	(no_connect
+		(at 209.55 91.44)
+	)
+	(no_connect
+		(at 184.15 91.44)
+	)
+	(no_connect
+		(at 184.15 63.5)
+	)
+	(no_connect
+		(at 209.55 96.52)
+	)
+	(no_connect
+		(at 209.55 68.58)
+	)
+	(no_connect
+		(at 184.15 88.9)
+	)
+	(no_connect
+		(at 209.55 78.74)
+	)
+	(no_connect
+		(at 196.85 106.68)
+	)
+	(no_connect
+		(at 209.55 63.5)
+	)
+	(no_connect
+		(at 194.31 53.34)
+	)
+	(no_connect
+		(at 184.15 93.98)
+	)
+	(no_connect
+		(at 209.55 88.9)
+	)
+	(no_connect
+		(at 209.55 81.28)
+	)
+	(no_connect
+		(at 209.55 99.06)
+	)
+	(no_connect
+		(at 184.15 96.52)
+	)
+	(no_connect
+		(at 199.39 53.34)
+	)
+	(no_connect
+		(at 184.15 66.04)
+	)
+	(no_connect
+		(at 184.15 86.36)
+	)
+	(no_connect
+		(at 209.55 83.82)
+	)
+	(no_connect
+		(at 209.55 73.66)
+	)
 	(wire
 		(pts
@@
 	(wire
 		(pts
-			(xy 179.07 74.93) (xy 179.07 76.2)
+			(xy 228.6 85.09) (xy 237.49 85.09)
+		)
+		(stroke
+			(width 0)
+			(type default)
+		)
+	)
+	(wire
+		(pts
+			(xy 177.8 74.93) (xy 177.8 76.2)
+		)
+		(stroke
+			(width 0)
+			(type default)
+		)
+	)
+	(wire
+		(pts
+			(xy 228.6 85.09) (xy 217.17 85.09)
 		)
 		(stroke
@@
 	(wire
 		(pts
-			(xy 228.6 86.36) (xy 228.6 88.9)
-		)
-		(stroke
-			(width 0)
-			(type default)
-		)
-	)
-	(wire
-		(pts
-			(xy 173.99 74.93) (xy 179.07 74.93)
+			(xy 228.6 81.28) (xy 228.6 85.09)
+		)
+		(stroke
+			(width 0)
+			(type default)
+		)
+	)
+	(wire
+		(pts
+			(xy 173.99 74.93) (xy 177.8 74.93)
 		)
 		(stroke
@@
 	(wire
 		(pts
-			(xy 181.61 106.68) (xy 181.61 83.82)
-		)
-		(stroke
-			(width 0)
-			(type default)
-		)
-	)
-	(wire
-		(pts
-			(xy 228.6 86.36) (xy 237.49 86.36)
+			(xy 228.6 85.09) (xy 228.6 88.9)
+		)
+		(stroke
+			(width 0)
+			(type default)
+		)
+	)
+	(wire
+		(pts
+			(xy 180.34 106.68) (xy 180.34 83.82)
 		)
 		(stroke
@@
 	(wire
 		(pts
+			(xy 237.49 85.09) (xy 237.49 86.36)
+		)
+		(stroke
+			(width 0)
+			(type default)
+		)
+	)
+	(wire
+		(pts
 			(xy 173.99 54.61) (xy 180.34 54.61)
 		)
@@
 	(wire
 		(pts
-			(xy 228.6 74.93) (xy 237.49 74.93)
-		)
-		(stroke
-			(width 0)
-			(type default)
-		)
-	)
-	(wire
-		(pts
-			(xy 179.07 76.2) (xy 184.15 76.2)
+			(xy 177.8 76.2) (xy 184.15 76.2)
 		)
 		(stroke
@@
 	(wire
 		(pts
-			(xy 173.99 106.68) (xy 181.61 106.68)
+			(xy 173.99 106.68) (xy 180.34 106.68)
 		)
 		(stroke
@@
 	(wire
 		(pts
+			(xy 217.17 86.36) (xy 209.55 86.36)
+		)
+		(stroke
+			(width 0)
+			(type default)
+		)
+	)
+	(wire
+		(pts
 			(xy 152.4 106.68) (xy 158.75 106.68)
 		)
@@
 	(wire
 		(pts
+			(xy 217.17 85.09) (xy 217.17 86.36)
+		)
+		(stroke
+			(width 0)
+			(type default)
+		)
+	)
+	(wire
+		(pts
 			(xy 152.4 54.61) (xy 158.75 54.61)
 		)
@@
 	(wire
 		(pts
-			(xy 209.55 86.36) (xy 228.6 86.36)
-		)
-		(stroke
-			(width 0)
-			(type default)
-		)
-	)
-	(wire
-		(pts
 			(xy 152.4 106.68) (xy 152.4 115.57)
 		)
@@
 	(wire
 		(pts
-			(xy 228.6 67.31) (xy 228.6 48.26)
+			(xy 228.6 66.04) (xy 228.6 48.26)
 		)
 		(stroke
@@
 	(wire
 		(pts
-			(xy 181.61 83.82) (xy 184.15 83.82)
+			(xy 228.6 73.66) (xy 237.49 73.66)
+		)
+		(stroke
+			(width 0)
+			(type default)
+		)
+	)
+	(wire
+		(pts
+			(xy 180.34 83.82) (xy 184.15 83.82)
 		)
 		(stroke
@@
 	(wire
 		(pts
-			(xy 237.49 85.09) (xy 237.49 86.36)
-		)
-		(stroke
-			(width 0)
-			(type default)
-		)
-	)
-	(wire
-		(pts
-			(xy 228.6 82.55) (xy 228.6 86.36)
+			(xy 237.49 83.82) (xy 237.49 85.09)
 		)
 		(stroke
@@
 	(symbol
 		(lib_id "Device:R")
-		(at 228.6 71.12 180)
+		(at 228.6 69.85 180)
 		(unit 1)
 		(body_style 1)
@@
 		(fields_autoplaced yes)
 		(property "Reference" "R8"
-			(at 231.14 69.8499 0)
+			(at 231.14 68.5799 0)
 			(show_name no)
 			(do_not_autoplace no)
@@
 		)
 		(property "Value" "1K"
-			(at 231.14 72.3899 0)
+			(at 231.14 71.1199 0)
 			(show_name no)
 			(do_not_autoplace no)
@@
 		)
 		(property "Footprint" "Resistor_THT:R_Axial_DIN0207_L6.3mm_D2.5mm_P10.16mm_Horizontal"
-			(at 230.378 71.12 90)
+			(at 230.378 69.85 90)
 			(hide yes)
 			(show_name no)
@@
 		)
 		(property "Datasheet" ""
-			(at 228.6 71.12 0)
+			(at 228.6 69.85 0)
 			(hide yes)
 			(show_name no)
@@
 		)
 		(property "Description" "Resistor"
-			(at 228.6 71.12 0)
+			(at 228.6 69.85 0)
 			(hide yes)
 			(show_name no)
@@
 	(symbol
 		(lib_id "Switch:SW_Push")
-		(at 237.49 80.01 270)
+		(at 237.49 78.74 270)
 		(unit 1)
 		(body_style 1)
@@
 		(fields_autoplaced yes)
 		(property "Reference" "SW2"
-			(at 241.3 78.7399 90)
+			(at 241.3 77.4699 90)
 			(show_name no)
 			(do_not_autoplace no)
@@
 		)
 		(property "Value" "SW_Push"
-			(at 241.3 81.2799 90)
+			(at 241.3 80.0099 90)
 			(show_name no)
 			(do_not_autoplace no)
@@
 		)
 		(property "Footprint" "Button_Switch_THT:SW_PUSH_6mm"
-			(at 242.57 80.01 0)
+			(at 242.57 78.74 0)
 			(hide yes)
 			(show_name no)
@@
 		)
 		(property "Datasheet" ""
-			(at 242.57 80.01 0)
+			(at 242.57 78.74 0)
 			(hide yes)
 			(show_name no)
@@
 		)
 		(property "Description" "Push button switch, generic, two pins"
-			(at 237.49 80.01 0)
+			(at 237.49 78.74 0)
 			(hide yes)
 			(show_name no)
@@
 	(symbol
 		(lib_id "Device:R")
-		(at 228.6 78.74 180)
+		(at 228.6 77.47 180)
 		(unit 1)
 		(body_style 1)
@@
 		(fields_autoplaced yes)
 		(property "Reference" "R9"
-			(at 231.14 77.4699 0)
+			(at 231.14 76.1999 0)
 			(show_name no)
 			(do_not_autoplace no)
@@
 		)
 		(property "Value" "1K"
-			(at 231.14 80.0099 0)
+			(at 231.14 78.7399 0)
 			(show_name no)
 			(do_not_autoplace no)
@@
 		)
 		(property "Footprint" "Resistor_THT:R_Axial_DIN0207_L6.3mm_D2.5mm_P10.16mm_Horizontal"
-			(at 230.378 78.74 90)
+			(at 230.378 77.47 90)
 			(hide yes)
 			(show_name no)
@@
 		)
 		(property "Datasheet" ""
-			(at 228.6 78.74 0)
+			(at 228.6 77.47 0)
 			(hide yes)
 			(show_name no)
@@
 		)
 		(property "Description" "Resistor"
-			(at 228.6 78.74 0)
-			(hide yes)
-			(show_name no)
+			(at 228.6 77.47 0)
+			(hide yes)
+			(show_name no)
