File: Wuerfel_Schaltplan/Wuerfel_Schaltplan.kicad_sch (KiCad schematic)
At the start: 21 parts, among them SW1 SW_Push, SW2 SW_Push

Commit message: Fix: Change Resitorvalues
Parts:
- R1, R2, R3, R4, R5, R6, R7: value 220 -> 330
Changed lines of the file:
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@@
 			)
 		)
-		(property "Value" "220"
+		(property "Value" "330"
 			(at 170.18 71.12 90)
 			(show_name no)
@@
 			)
 		)
-		(property "Value" "220"
+		(property "Value" "330"
 			(at 170.18 60.96 90)
 			(show_name no)
@@
 			)
 		)
-		(property "Value" "220"
+		(property "Value" "330"
 			(at 170.18 50.8 90)
 			(show_name no)
@@
 			)
 		)
-		(property "Value" "220"
+		(property "Value" "330"
 			(at 170.18 81.28 90)
 			(show_name no)
@@
 			)
 		)
-		(property "Value" "220"
+		(property "Value" "330"
 			(at 170.18 40.64 90)
 			(show_name no)
@@
 			)
 		)
-		(property "Value" "220"
+		(property "Value" "330"
 			(at 170.18 102.87 90)
 			(show_name no)
@@
 			)
 		)
-		(property "Value" "220"
+		(property "Value" "330"
 			(at 170.18 91.44 90)
 			(show_name no)
